File: schematic/schematic.sch (EAGLE design)
At the start: 5 parts, among them IC1 74LS164N, IC2 74LS164N, X1 RS232

Commit message: Slight modifications
Connections:
- net GND: now also X1.5
Changed lines of the file:
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@@
 <setting verticaltext="up"/>
 </settings>
-<grid distance="0.1" unitdist="inch" unit="inch" style="dots" multiple="1" display="yes" altdistance="0.01" altunitdist="inch" altunit="inch"/>
+<grid distance="0.1" unitdist="inch" unit="inch" style="lines" multiple="1" display="no" altdistance="0.01" altunitdist="inch" altunit="inch"/>
 <layers>
 <layer number="1" name="Top" color="4" fill="1" visible="no" active="no"/>
@@
 <part name="X1" library="con-subd" deviceset="F09" device="H" value="RS232"/>
 <part name="ZX1" library="con-3m" deviceset="228-?00-0602J" device="1277-" value="ZIF28"/>
+<part name="GND3" library="supply1" deviceset="GND" device=""/>
 </parts>
 <sheets>
@@
 <instance part="X1" gate="G$1" x="43.18" y="60.96" rot="R180"/>
 <instance part="ZX1" gate="G$1" x="175.26" y="50.8"/>
+<instance part="GND3" gate="1" x="53.34" y="53.34"/>
 </instances>
 <busses>
@@
 <net name="N$2" class="0">
 <segment>
-<wire x1="119.38" y1="2.54" x2="119.38" y2="30.48" width="0.1524" layer="91"/>
+<wire x1="119.38" y1="22.86" x2="119.38" y2="30.48" width="0.1524" layer="91"/>
 <pinref part="IC2" gate="A" pin="CLR"/>
 <wire x1="119.38" y1="30.48" x2="124.46" y2="30.48" width="0.1524" layer="91"/>
@@
 <pinref part="MCU1" gate="G$1" pin="RST@2"/>
 <wire x1="68.58" y1="45.72" x2="60.96" y2="45.72" width="0.1524" layer="91"/>
-<wire x1="60.96" y1="45.72" x2="60.96" y2="2.54" width="0.1524" layer="91"/>
-<wire x1="60.96" y1="2.54" x2="119.38" y2="2.54" width="0.1524" layer="91"/>
+<wire x1="60.96" y1="45.72" x2="60.96" y2="22.86" width="0.1524" layer="91"/>
+<wire x1="60.96" y1="22.86" x2="119.38" y2="22.86" width="0.1524" layer="91"/>
 </segment>
 </net>
@@
 <pinref part="ZX1" gate="G$1" pin="14"/>
 </segment>
+<segment>
+<pinref part="X1" gate="G$1" pin="5"/>
+<pinref part="GND3" gate="1" pin="GND"/>
+<wire x1="50.8" y1="66.04" x2="53.34" y2="66.04" width="0.1524" layer="91"/>
+<wire x1="53.34" y1="66.04" x2="53.34" y2="55.88" width="0.1524" layer="91"/>
+</segment>
 </net>
